Commit message: new model.

File: barret_hand_defs/defs/barret_hand.urdf.xacro (robot description, xacro)
@@ -31,7 +31,4 @@
     <xacro:property name="highResModelDirectory" value="${homeDirectory}/meshes/splitModels" />
     <xacro:property name="PI" value="3.1415926535897931" />
-    <material name="DarpaGrey">
-        <color rgba="0.9 0.9 0.9 1.0"/>
-    </material>
     <xacro:macro name="palm" params="prefix parent">
         <link name="${prefix}_HandPalmLink" >
@@ -44,8 +41,7 @@
         </inertial>
         <visual>
-            <material name="DarpaGrey" />
-            <origin xyz="0 0 0" rpy="0 0 0" />
+            <origin xyz="0 0 0" rpy="${PI} 0 0" />
             <geometry>
-                    <mesh filename="${homeDirectory}/meshes/palm.DAE"/>
+                    <mesh filename="${homeDirectory}/meshes/HandPalmLink.dae"/>
             </geometry>
         </visual>
@@ -60,5 +56,5 @@
             <parent link="${parent}"/>
             <child link="${prefix}_HandPalmLink"/>
-            <origin xyz="0 0 0.04" rpy="0 0 -${0.5 * PI}"/>
+            <origin xyz="0.0 0 0.0" rpy="0 0 0"/>
             <provideFeedback value="true"/>
         </joint>
@@ -67,8 +63,7 @@
         <link name="${prefix}_HandFinger${number}KnuckleOneLink">
         <visual>
-            <material name="DarpaGrey" />
-            <origin xyz="0 0 0" rpy="${0.5 * PI} 0 -${0.5 * PI}" />
+            <origin xyz="0 0 -0.017" rpy="${0.5 * PI} 0 -${0.5 * PI}" />
             <geometry>
-                <mesh filename="${homeDirectory}/meshes/firstFingerLink.DAE"/>
+                <mesh filename="${homeDirectory}/meshes/KnuckleOneLink.dae"/>
             </geometry>
         </visual>
@@ -83,5 +78,5 @@
             <origin xyz="0 0 0" rpy="${0.5 * PI} 0 -${0.5 * PI}" />
             <geometry>
-            <mesh filename="${homeDirectory}/meshes/firstFingerLink.stl"/>
+                    <mesh filename="${homeDirectory}/meshes/firstFingerLink.stl"/>
             </geometry>
             <mu1 value="50000.0" />
@@ -97,5 +92,5 @@
             <axis xyz="${axis}"/>
             <limit effort="1" lower="0" upper="${PI}" velocity="3.27"/>
-            <dynamics damping="0.005" friction="100.0"/>
+            <dynamics damping="0.05" friction="100.0"/>
         </joint>
     </xacro:macro>
@@ -103,8 +98,7 @@
         <link name="${prefix}_HandFinger${number}KnuckleTwoLink">
             <visual>
-                <material name="DarpaGrey" />
                 <origin xyz="0 0 0" rpy="${PI} ${0.5 * PI} 0" />
                 <geometry>
-                    <mesh filename="${homeDirectory}/meshes/secondFingerLink.DAE"/>
+                    <mesh filename="${homeDirectory}/meshes/KnuckleTwoLink.dae"/>
                 </geometry>
             </visual>
@@ -140,8 +134,7 @@
         <link name="${prefix}_HandFinger${number}KnuckleThreeLink">
           <visual>
-            <material name="DarpaGrey" />
             <origin xyz="0 0 0" rpy="0 ${0.5 * PI} 0" />
             <geometry>
-                <mesh filename="${homeDirectory}/meshes/thirdFingerLink.DAE"/>
+                <mesh filename="${homeDirectory}/meshes/KnuckleThreeLink.dae"/>
             </geometry>
           </visual>
@@ -156,5 +149,5 @@
             <origin xyz="0 0 0" rpy="0 ${0.5 * PI} 0" />
             <geometry>
-              <mesh filename="${homeDirectory}/meshes/thirdFingerLink.stl"/>
+                    <mesh filename="${homeDirectory}/meshes/thirdFingerLink.stl"/>
             </geometry>
             <mu1 value="50000.0" />
