Commit message: switched to catkin and Orocos

File: barrett_hand_defs/defs/barret_hand.urdf.xacro (robot description, xacro)
@@ -28,5 +28,5 @@
        xmlns:interface="http://playerstage.sourceforge.net/gazebo/xmlschema/#interface"
        xmlns:xacro="http://www.ros.org/wiki/xacro">
-    <xacro:property name="homeDirectory" value="package://barret_hand_defs" />
+    <xacro:property name="homeDirectory" value="package://barrett_hand_defs" />
     <xacro:property name="highResModelDirectory" value="${homeDirectory}/meshes/splitModels" />
     <xacro:property name="PI" value="3.1415926535897931" />

Commit message: velma integration

File: barrett_hand_defs/defs/barret_hand.urdf.xacro (robot description, xacro)
@@ -31,5 +31,5 @@
     <xacro:property name="highResModelDirectory" value="${homeDirectory}/meshes/splitModels" />
     <xacro:property name="PI" value="3.1415926535897931" />
-    <xacro:macro name="palm" params="prefix parent">
+    <xacro:macro name="palm" params="prefix parent *origin">
         <link name="${prefix}_HandPalmLink" >
         <inertial>
@@ -56,5 +56,6 @@
             <parent link="${parent}"/>
             <child link="${prefix}_HandPalmLink"/>
-            <origin xyz="0.0 0 0.0" rpy="0 0 0"/>
+            <insert_block name="origin"/>
+<!--            <origin xyz="0.0 0 0.0" rpy="0 0 0"/>-->
             <provideFeedback value="true"/>
         </joint>
@@ -172,6 +173,8 @@
         <xacro:KnuckleThree prefix="${prefix}" number="${number}"/>
     </xacro:macro>
-    <xacro:macro name="barret_hand" params="prefix parent">
-        <xacro:palm prefix="${prefix}" parent="${parent}"/>
+    <xacro:macro name="barret_hand" params="prefix parent *origin">
+        <xacro:palm prefix="${prefix}" parent="${parent}">
+            <insert_block name="origin"/>
+        </xacro:palm>
         <xacro:fingers prefix="${prefix}" parent="${prefix}_HandPalmLink" number="Three" xyz="0 -0.05 0.0801966" rpy="-${0.5 * PI} -0.0429350996 -${0.5 * PI}"/>
         <xacro:KnuckleOne prefix="${prefix}" number="One" xyz=".02497 0 0.0587966" rpy="0 0 ${0.5 * PI}" axis="0 0 -1"/>

Commit message: add gravity falg for gazebo.

File: barrett_hand_defs/defs/barret_hand.urdf.xacro (robot description, xacro)
@@ -53,9 +53,11 @@
             </collision>
         </link>
+        <gazebo reference="${prefix}_HandPalmLink">
+          <turnGravityOff>true</turnGravityOff>
+        </gazebo>
         <joint name="${prefix}_HandPalmJoint" type="fixed">
             <parent link="${parent}"/>
             <child link="${prefix}_HandPalmLink"/>
             <insert_block name="origin"/>
-<!--            <origin xyz="0.0 0 0.0" rpy="0 0 0"/>-->
             <provideFeedback value="true"/>
         </joint>
@@ -87,4 +89,7 @@
         </collision>
         </link>
+        <gazebo reference="${prefix}_HandFinger${number}KnuckleOneLink">
+          <turnGravityOff>true</turnGravityOff>
+        </gazebo>
         <joint name="${prefix}_HandFinger${number}KnuckleOneJoint" type="revolute">
             <parent link="${prefix}_HandPalmLink"/>
@@ -122,4 +127,7 @@
             </collision>
         </link>
+        <gazebo reference="${prefix}_HandFinger${number}KnuckleTwoLink">
+          <turnGravityOff>true</turnGravityOff>
+        </gazebo>
         <joint name="${prefix}_HandFinger${number}KnuckleTwoJoint" type="revolute">
             <parent link="${parent}"/>
@@ -158,4 +166,7 @@
           </collision>
         </link>
+        <gazebo reference="${prefix}_HandFinger${number}KnuckleThreeLink">
+          <turnGravityOff>true</turnGravityOff>
+        </gazebo>
         <joint name="${prefix}_HandFinger${number}KnuckleThreeJoint" type="revolute">
             <parent link="${prefix}_HandFinger${number}KnuckleTwoLink"/>

Commit message: added collision description

File: barrett_hand_defs/defs/barret_hand.urdf.xacro (robot description, xacro)
@@ -33,5 +33,5 @@
     <xacro:macro name="palm" params="prefix parent *origin">
         <link name="${prefix}_HandPalmLink" >
-        <inertial>
+          <inertial>
             <origin xyz="0.00035500 -0.00499005 0.04864979" />
             <mass value="0.63352875" />
@@ -39,17 +39,52 @@
                                        iyy="0.00080944"  iyz="-0.00014417"
                                                          izz="0.00068788" />
-        </inertial>
-        <visual>
+          </inertial>
+          <visual>
             <origin xyz="0 0 0" rpy="${PI} 0 0" />
             <geometry>
                     <mesh filename="${homeDirectory}/meshes/HandPalmLink.dae"/>
             </geometry>
-        </visual>
-            <collision>
+          </visual>
+          <collision>
             <origin xyz="0 0 0" rpy="0 0 0" />
             <geometry>
-                    <mesh filename="${homeDirectory}/meshes/palm.stl"/>
-            </geometry>
-            </collision>
+              <mesh filename="${homeDirectory}/meshes/palm.stl"/>
+            </geometry>
+          </collision>
+          <self_collision_checking>
+            <origin xyz="0 0 0.03" rpy="0 0 0"/>
+            <geometry>
+              <capsule radius="0.05" length="0.06"/>
+            </geometry>
+          </self_collision_checking>
+          <self_collision_checking>
+            <origin xyz="-0.05 0 -0.05" rpy="0 0.785375 0"/>
+            <geometry>
+              <capsule radius="0.05" length="0.06"/>
+            </geometry>
+          </self_collision_checking>
+          <self_collision_checking>
+            <origin xyz="0 0 0" rpy="0 0 0"/>
+            <geometry>
+              <convex>
+                <!-- fingers' base links -->
+                <point xyz="0.06 0 0" frame="${prefix}_HandFingerOneKnuckleOneLink"/>
+                <point xyz="0.06 0 0" frame="${prefix}_HandFingerTwoKnuckleOneLink"/>
+                <point xyz="0 -0.06 0.06" frame="${prefix}_HandPalmLink"/>
+                <!-- proximal fingers' links -->
+<!--                <point xyz="0 0 0" frame="${prefix}_HandFingerOneKnuckleTwoLink"/>
+                <point xyz="0 0 0" frame="${prefix}_HandFingerTwoKnuckleTwoLink"/>
+                <point xyz="0 0 0" frame="${prefix}_HandFingerThreeKnuckleTwoLink"/>
+-->
+                <!-- distal fingers' links -->
+                <point xyz="0 0 0" frame="${prefix}_HandFingerOneKnuckleThreeLink"/>
+                <point xyz="0 0 0" frame="${prefix}_HandFingerTwoKnuckleThreeLink"/>
+                <point xyz="0 0 0" frame="${prefix}_HandFingerThreeKnuckleThreeLink"/>
+                <point xyz="0.06 0 0" frame="${prefix}_HandFingerOneKnuckleThreeLink"/>
+                <point xyz="0.06 0 0" frame="${prefix}_HandFingerTwoKnuckleThreeLink"/>
+                <point xyz="0.06 0 0" frame="${prefix}_HandFingerThreeKnuckleThreeLink"/>
+              </convex>
+            </geometry>
+          </self_collision_checking>
         </link>
         <gazebo reference="${prefix}_HandPalmLink">

Commit message: collision model

File: barrett_hand_defs/defs/barret_hand.urdf.xacro (robot description, xacro)
@@ -53,9 +53,10 @@
           </collision>
           <self_collision_checking>
-            <origin xyz="0 0 0.03" rpy="0 0 0"/>
-            <geometry>
-              <capsule radius="0.05" length="0.06"/>
+            <origin xyz="0 0 0.04" rpy="0 0 0"/>
+            <geometry>
+              <capsule radius="0.05" length="0.04"/>
             </geometry>
           </self_collision_checking>
+<!--
           <self_collision_checking>
             <origin xyz="-0.05 0 -0.05" rpy="0 0.785375 0"/>
@@ -64,4 +65,5 @@
             </geometry>
           </self_collision_checking>
+-->
           <self_collision_checking>
             <origin xyz="0 0 0" rpy="0 0 0"/>

Commit message: modified xarco

File: barrett_hand_defs/defs/barret_hand.urdf.xacro (robot description, xacro)
@@ -52,15 +52,9 @@
             </geometry>
           </collision>
+<!--
           <self_collision_checking>
             <origin xyz="0 0 0.04" rpy="0 0 0"/>
             <geometry>
               <capsule radius="0.05" length="0.04"/>
-            </geometry>
-          </self_collision_checking>
-<!--
-          <self_collision_checking>
-            <origin xyz="-0.05 0 -0.05" rpy="0 0.785375 0"/>
-            <geometry>
-              <capsule radius="0.05" length="0.06"/>
             </geometry>
           </self_collision_checking>
@@ -70,4 +64,9 @@
             <geometry>
               <convex>
+                <!-- gripper base points -->
+                <point xyz="0.03 0.03 0.0" frame="${prefix}_HandPalmLink"/>
+                <point xyz="-0.03 0.03 0.0" frame="${prefix}_HandPalmLink"/>
+                <point xyz="-0.03 -0.03 0.0" frame="${prefix}_HandPalmLink"/>
+                <point xyz="0.03 -0.03 0.0" frame="${prefix}_HandPalmLink"/>
                 <!-- fingers' base links -->
                 <point xyz="0.06 0 0" frame="${prefix}_HandFingerOneKnuckleOneLink"/>
